File: KiCad/LargeKickstarter/LargeKickstarter.kicad_pcb (KiCad board)
At the start: 2 copper layers, 398.2 x 398.2 mm, 1578 parts, among them M2 MountingHole_2-5mm, M3 MountingHole_2-5mm, P1 CONN_01X03, P2 CONN_01X02, P3 CONN_01X05, P4 CONN_02X03, P5 CONN_01X06, SW1 HOUR, SW2 MIN, SW4 SOFT, U1 HT16K33, U10 HT16K33, U11 HT16K33_BOUT, U12 HT16K33, U2 DS3231, U3 ATMEGA328-TQFP, U4 HT16K33, U5 HT16K33_BOUT, U6 HT16K33_BOUT, U7 Arduino_Nano, U8 UNO_FOOTPRINT, U9 HT16K33_BOUT

Commit message: Further tweaks
Added PTH components for power section and buttons. Fixed some
disconnects.
Parts:
- added D6: DIODE, Diodes_ThroughHole:Diode_DO-41_SOD81_Horizontal_RM10, F.Cu at (91.2, 349.3)
- added R18: 10K, Resistors_ThroughHole:Resistor_Horizontal_RM10mm, F.Cu at (25.2, 383.4)
- added R19: 10K, Resistors_ThroughHole:Resistor_Horizontal_RM10mm, F.Cu at (25.2, 402.7)
- added R20: 10K, Resistors_ThroughHole:Resistor_Horizontal_RM10mm, F.Cu at (25.2, 406.5)
- C1, C4, C5, C6, C7, C8: footprint LikeClockwork:capacitor_0603 -> Capacitors_SMD:C_0603_HandSoldering
- D2, D3, D4, D5: footprint LikeClockwork:signal_diode -> Diodes_SMD:SOD-323
- P2: footprint LikeClockwork:POWER_IN -> Pin_Headers:Pin_Header_Straight_1x02
- R1, R10, R11, R12, R13, R14, R15, R16, R17, R2, R3, R4, R5, R6, R7, R8, R9: footprint LikeClockwork:resistor_0603 -> Resistors_SMD:R_0603_HandSoldering
- U2: footprint LikeClockwork:DS3231 -> Housings_SOIC:SOIC-16_7.5x10.3mm_Pitch1.27mm
Connections:
- net Vcc renamed VCC
- P3 pad N/C: (no net) -> Net-(P3-PadN/C)
- P5 pad 1: (no net) -> Net-(P5-Pad1)
- P5 pad 2: (no net) -> Net-(P5-Pad2)
- U2 pad 1: (no net) -> Net-(U2-Pad1)
- U2 pad 3: (no net) -> Net-(U2-Pad3)
- U2 pad 4: (no net) -> Net-(U2-Pad4)
- U3 pad 7: (no net) -> Net-(U3-Pad7)
- U3 pad 8: (no net) -> Net-(U3-Pad8)
- U8 pad 1: (no net) -> Net-(U8-Pad1)
- U8 pad 2: (no net) -> Net-(U8-Pad2)
Routing:
- net 7: track 334.9 -> 343.1 mm
- net RAW: track 10.7 -> 15.0 mm
- net COM-0-7: track 502.6 -> 506.8 mm
- net 6: track 313.1 -> 316.7 mm
- net 5: track 293.3 -> 296.9 mm
- net COM-2-7: track 562.9 -> 564.5 mm
- net Vin: track 172.2 -> 172.8 mm
